Commit message: Add Gazebo Harmonic camera sensor with ROS image output

File: src/gazebo_micro_bot/urdf/micro_bot.urdf (robot description, URDF)
Before this commit: robot micro_bot, 3 links, 2 joints
Links:
- added link camera_link; visual box size=0.05 0.05 0.05
Joints:
- added joint camera_joint: type fixed, parent base_link, child camera_link, origin xyz=0.15 0 0.15 rpy=0 0 0

Commit message: Add Gazebo Harmonic LiDAR publishing /scan

File: src/gazebo_micro_bot/urdf/micro_bot.urdf (robot description, URDF)
Before this commit: robot micro_bot, 4 links, 3 joints
Links:
- added link lidar_link; visual cylinder length=0.05 radius=0.03
Joints:
- added joint lidar_joint: type fixed, parent base_link, child lidar_link, origin xyz=0.2 0 0.18 rpy=0 0 0
